File: PCB/EEGamp/EEGamp.sch (KiCad schematic (older format))
At the start: 100 parts, among them J1 Conn_02x17, Q1 BC847, Q2 BC847, Q3 BC847, Q4 BC847, Q5 BC857, Q6 BC857, Q7 BC857, Q8 BC857, U1 TLC277, U2 AD620, U3 AD620, U4 TLC277, U5 TLC277, U6 TLC277

Commit message: Test points added
Parts:
- added TP1: CH2, TestPoint:TestPoint_2Pads_Pitch2.54mm_Drill0.8mm, symbol Connector:TestPoint_2Pole
- added TP2: CH1, TestPoint:TestPoint_2Pads_Pitch2.54mm_Drill0.8mm, symbol Connector:TestPoint_2Pole
- added TP3: R_LEG, TestPoint:TestPoint_Loop_D1.80mm_Drill1.0mm_Beaded, symbol Connector:TestPoint
- added TP4: DC Check CH2, TestPoint:TestPoint_Loop_D1.80mm_Drill1.0mm_Beaded, symbol Connector:TestPoint
- added TP5: DC Check CH1, TestPoint:TestPoint_Loop_D1.80mm_Drill1.0mm_Beaded, symbol Connector:TestPoint
- added TP6: CalGND, TestPoint:TestPoint_Loop_D1.80mm_Drill1.0mm_Beaded, symbol Connector:TestPoint
- added TP7: CalU, TestPoint:TestPoint_Loop_D1.80mm_Drill1.0mm_Beaded, symbol Connector:TestPoint
- U4, U5, U6: footprint (none) -> Package_SO:SOIC-8_3.9x4.9mm_P1.27mm
Connections:
- net CH1+: now also TP2.2
- net CH1-: now also TP2.1
- net CH2+: now also TP1.2
- net CH2-: now also TP1.1
- net R_LEG: now also TP3.1
- net at C15.2, U2.6: now also TP4.1
- net at C16.2, U3.6: now also TP5.1
- net at R32.2: now also TP6.1
- net at R33.2: now also TP7.1
- no-connect marks 11 -> 2
Changed lines of the file:
@@
 	1    0    0    -1
 $EndComp
-NoConn ~ 1450 1700
-NoConn ~ 1450 3100
 Wire Wire Line
 	3000 2900 3250 2900
@@
 	1    0    0    -1
 $EndComp
-NoConn ~ 1450 4450
-NoConn ~ 1450 5850
 Wire Wire Line
 	3000 5650 3250 5650
@@
 Wire Wire Line
 	1450 7550 1950 7550
-NoConn ~ 1450 7550
 Text Label 1450 7550 0    50   ~ 0
 R_LEG
@@
 	8950 2500 8750 2500
 Connection ~ 8950 3000
-NoConn ~ 6300 1750
 Wire Wire Line
 	5800 2400 6300 2400
@@
 	8950 5250 8750 5250
 Connection ~ 8950 5750
-NoConn ~ 6300 4500
 Wire Wire Line
 	5800 5150 6300 5150
@@
 	0    1    1    0
 $EndComp
-NoConn ~ 9750 8000
-NoConn ~ 9750 8500
 Wire Wire Line
 	9750 8000 10250 8000
@@
 F 0 "U4" H 5108 6896 50  0000 L CNN
 F 1 "TLC277" H 5108 6805 50  0000 L CNN
-F 2 "" H 5150 6850 50  0001 C CNN
+F 2 "Package_SO:SOIC-8_3.9x4.9mm_P1.27mm" H 5150 6850 50  0001 C CNN
 F 3 "http://www.ti.com/lit/ds/symlink/tlc272.pdf" H 5150 6850 50  0001 C CNN
 	3    5150 6850
@@
 F 0 "U6" H 11650 6050 50  0000 L CNN
 F 1 "TLC277" H 11650 5950 50  0000 L CNN
-F 2 "" H 11950 5950 50  0001 C CNN
+F 2 "Package_SO:SOIC-8_3.9x4.9mm_P1.27mm" H 11950 5950 50  0001 C CNN
 F 3 "http://www.ti.com/lit/ds/symlink/tlc272.pdf" H 11950 5950 50  0001 C CNN
 	3    11950 5950
@@
 F 0 "U5" H 11750 3300 50  0000 L CNN
 F 1 "TLC277" H 11750 3200 50  0000 L CNN
-F 2 "" H 12050 3200 50  0001 C CNN
+F 2 "Package_SO:SOIC-8_3.9x4.9mm_P1.27mm" H 12050 3200 50  0001 C CNN
 F 3 "http://www.ti.com/lit/ds/symlink/tlc272.pdf" H 12050 3200 50  0001 C CNN
 	3    12050 3200
@@
 	11950 2900 11950 2850
 Connection ~ 11950 2850
+$Comp
+L Connector:TestPoint_2Pole TP1
+U 1 1 5C9CF83E
+P 1450 2400
+F 0 "TP1" V 1200 2250 50  0000 L CNN
+F 1 "CH2" V 1700 2250 50  0000 L CNN
+F 2 "TestPoint:TestPoint_2Pads_Pitch2.54mm_Drill0.8mm" H 1450 2400 50  0001 C CNN
+F 3 "~" H 1450 2400 50  0001 C CNN
+	1    1450 2400
+	0    1    1    0
+$EndComp
+Wire Wire Line
+	1450 1700 1450 2200
+Wire Wire Line
+	1450 2600 1450 3100
+$Comp
+L Connector:TestPoint_2Pole TP2
+U 1 1 5CA29D1B
+P 1450 5150
+F 0 "TP2" V 1200 5000 50  0000 L CNN
+F 1 "CH1" V 1700 5000 50  0000 L CNN
+F 2 "TestPoint:TestPoint_2Pads_Pitch2.54mm_Drill0.8mm" H 1450 5150 50  0001 C CNN
+F 3 "~" H 1450 5150 50  0001 C CNN
+	1    1450 5150
+	0    1    1    0
+$EndComp
+Wire Wire Line
+	1450 4450 1450 4950
+Wire Wire Line
+	1450 5350 1450 5850
+$Comp
+L Connector:TestPoint TP4
+U 1 1 5CAFF7BF
+P 6300 1750
+F 0 "TP4" H 6358 1870 50  0000 L CNN
+F 1 "DC Check CH2" H 6358 1779 50  0000 L CNN
+F 2 "TestPoint:TestPoint_Loop_D1.80mm_Drill1.0mm_Beaded" H 6500 1750 50  0001 C CNN
+F 3 "~" H 6500 1750 50  0001 C CNN
+	1    6300 1750
+	1    0    0    -1
+$EndComp
+$Comp
+L Connector:TestPoint TP6
+U 1 1 5CB3D2B3
+P 9750 8000
+F 0 "TP6" V 9945 8074 50  0000 C CNN
+F 1 "CalGND" V 9854 8074 50  0000 C CNN
+F 2 "TestPoint:TestPoint_Loop_D1.80mm_Drill1.0mm_Beaded" H 9950 8000 50  0001 C CNN
+F 3 "~" H 9950 8000 50  0001 C CNN
+	1    9750 8000
+	0    -1   -1   0
+$EndComp
+$Comp
+L Connector:TestPoint TP7
+U 1 1 5CB3D770
+P 9750 8500
+F 0 "TP7" V 9650 8600 50  0000 C CNN
+F 1 "CalU" V 9550 8600 50  0000 C CNN
+F 2 "TestPoint:TestPoint_Loop_D1.80mm_Drill1.0mm_Beaded" H 9950 8500 50  0001 C CNN
+F 3 "~" H 9950 8500 50  0001 C CNN
+	1    9750 8500
+	0    -1   -1   0
+$EndComp
+$Comp
+L Connector:TestPoint TP3
+U 1 1 5CB5F41E
+P 1450 7550
+F 0 "TP3" V 1645 7624 50  0000 C CNN
+F 1 "R_LEG" V 1554 7624 50  0000 C CNN
+F 2 "TestPoint:TestPoint_Loop_D1.80mm_Drill1.0mm_Beaded" H 1650 7550 50  0001 C CNN
+F 3 "~" H 1650 7550 50  0001 C CNN
+	1    1450 7550
+	0    -1   -1   0
+$EndComp
+$Comp
+L Connector:TestPoint TP5
+U 1 1 5CB7EC6C
+P 6300 4500
+F 0 "TP5" H 6358 4620 50  0000 L CNN
+F 1 "DC Check CH1" H 6358 4529 50  0000 L CNN
+F 2 "TestPoint:TestPoint_Loop_D1.80mm_Drill1.0mm_Beaded" H 6500 4500 50  0001 C CNN
+F 3 "~" H 6500 4500 50  0001 C CNN
+	1    6300 4500
+	1    0    0    -1
+$EndComp
 $EndSCHEMATC

Commit message: Project reborn! =]
Parts:
- removed J1: Conn_02x17, Connector_IDC:IDC-Header_2x17_P2.54mm_Horizontal_Lock, symbol Connector_Generic:Conn_02x17_Odd_Even
- removed Q1, Q2, Q3, Q4: BC847, Package_TO_SOT_SMD:SOT-23, symbol Transistor_BJT:BC847
- removed Q5, Q6, Q7, Q8: BC857, Package_TO_SOT_SMD:SOT-23, symbol Transistor_BJT:BC857
- removed TP1: CH2, TestPoint:TestPoint_2Pads_Pitch2.54mm_Drill0.8mm, symbol Connector:TestPoint_2Pole
- removed TP2: CH1, TestPoint:TestPoint_2Pads_Pitch2.54mm_Drill0.8mm, symbol Connector:TestPoint_2Pole
- removed TP3: R_LEG, TestPoint:TestPoint_Loop_D1.80mm_Drill1.0mm_Beaded, symbol Connector:TestPoint
- removed TP4: DC Check CH2, TestPoint:TestPoint_Loop_D1.80mm_Drill1.0mm_Beaded, symbol Connector:TestPoint
- removed TP5: DC Check CH1, TestPoint:TestPoint_Loop_D1.80mm_Drill1.0mm_Beaded, symbol Connector:TestPoint
- removed TP6: CalGND, TestPoint:TestPoint_Loop_D1.80mm_Drill1.0mm_Beaded, symbol Connector:TestPoint
- removed TP7: CalU, TestPoint:TestPoint_Loop_D1.80mm_Drill1.0mm_Beaded, symbol Connector:TestPoint
- removed U1, U4, U5, U6: TLC277, Package_SO:SOIC-8_3.9x4.9mm_P1.27mm, symbol Amplifier_Operational:TLC277
- removed U2: AD620, Package_SO:SOIC-8_3.9x4.9mm_P1.27mm, symbol Amplifier_Instrumentation:AD620
- added Q1, Q2, Q3, Q4: BC847, Package_TO_SOT_SMD:SOT-23, symbol Transistor_NPN:BC847
- added Q5, Q6, Q7, Q8: BC857, Package_TO_SOT_SMD:SOT-23, symbol Transistor_PNP:BC857
- added U1, U2, U5, U6: AD822, Package_SO:SOIC-8_3.9x4.9mm_P1.27mm, symbol Amplifier_Operational:AD822
- added U4: AD620, Package_SO:SOIC-8_3.9x4.9mm_P1.27mm, symbol Amplifier_Instrumentation:AD620
- added X1: CH2, Connector_Header:PinHeader_1x02_P2.54mm_Vertical, symbol Connector_Header:A2541WV-2P
- added X2: CH1, Connector_Header:PinHeader_1x02_P2.54mm_Vertical, symbol Connector_Header:A2541WV-2P
- added X3: R_LEG, Connector_Header:PinHeader_1x01_P2.54mm_Vertical, symbol Connector_Header:C81276
- added X4: Cal, Connector_Header:PinHeader_1x02_P2.54mm_Vertical, symbol Connector_Header:A2541WV-2P
- added X5: DC Check CH1, Connector_Header:PinHeader_1x01_P2.54mm_Vertical, symbol Connector_Header:C81276
- added X6: DC Check CH2, Connector_Header:PinHeader_1x01_P2.54mm_Vertical, symbol Connector_Header:C81276
- added X7: PIN_HEADER_2X17_2.54, Connector_Header:PinHeader_2x17_P2.54mm_Vertical, symbol Connector_Header:PIN_HEADER_2X17_2.54
- C1, C10, C11, C12, C13, C14, C15, C16, C17, C18, C19, C2, C20, C21, C22, C23, C24, C25, C26, C27, C28, C3, C30, C31, C32, C33, C34, C35, C4, C5, C6, C7, C8, C9: footprint Capacitor_SMD:C_0805_2012Metric_Pad1.15x1.40mm_HandSolder -> Capacitors:C_0603; symbol Device:C -> EEGamp-rescue:C-Device
- C29, C36: footprint Capacitor_Tantalum_SMD:CP_EIA-2012-15_AVX-P_Pad1.30x1.05mm_HandSolder -> Capacitors_Tantalum:CP_EIA-3528-15_AVX-H; symbol Device:CP -> EEGamp-rescue:CP-Device
- JP1, JP2, JP3, JP4, JP5, JP6: symbol Jumper:SolderJumper_2_Open -> EEGamp-rescue:SolderJumper_2_Open-Jumper
- R1, R10, R11, R12, R13, R14, R15, R16, R17, R18, R19, R2, R20, R21, R22, R23, R24, R25, R26, R27, R28, R29, R3, R30, R31, R32, R33, R34, R35, R36, R37, R38, R39, R4, R40, R5, R6, R7, R8, R9: footprint Resistor_SMD:R_0805_2012Metric_Pad1.15x1.40mm_HandSolder -> Resistors:R_0603; symbol Device:R_US -> EEGamp-rescue:R_US-Device
- RV1, RV2, RV3: footprint Potentiometer_THT:Potentiometer_Bourns_3296Y_Vertical -> Resistors:BOURNS_3296W_Vertical; symbol Device:R_POT_US -> EEGamp-rescue:R_POT_US-Device
Connections:
- net +5V: now also U1.8 (V+), U2.8 (V+), U4.7 (Vs+), U5.8 (V+)
- net 2.0V: now also Q1.2 (E), Q2.3 (C), Q3.2 (E), Q4.3 (C), Q5.3 (C), Q6.2 (E), Q7.3 (C), Q8.2 (E), U4.5 (Ref), U6.1, U6.3 (+), X7.3
- net ADIN0: now also U6.7
- net ADIN1: now also U5.7
- net CH1+: now also X2.1
- net CH1-: now also X2.2
- net CH2+: now also X1.1
- net CH2-: now also X1.2
- net COM: now also U1.6 (-)
- net GNDA: now also U1.4 (V-), U2.4 (V-), U4.4 (Vs-), U5.4 (V-), U6.4 (V-), X7.11, X7.13, X7.5, X7.7, X7.9
- net PWM: now also X7.30
- net R_LEG: now also X3.1
- net at R16.1: now also U3.1 (Rg)
- net at R11.1: now also U3.2 (-)
- net at R13.1: now also U3.3 (+)
- net at C15.2: now also U3.6, X5.1
- net at R17.1: now also U3.8 (Rg)
- net at C1.2, C6.2, R2.1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: now also Q2.2 (E), Q6.3 (C)
- net at C1.1, C5.1, R1.2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: now also Q1.3 (C), Q5.2 (E)
- net at R18.1: now also U4.1 (Rg); no longer U3.1 (Rg)
- net at R12.1: now also U4.2 (-); no longer U3.2 (-)
- net at R14.1: now also U4.3 (+); no longer U3.3 (+)
- net at C16.2: now also U4.6, X6.1; no longer U3.6
- net at R19.1: now also U4.8 (Rg); no longer U3.8 (Rg)
- net at C2.2, C8.2, R10.2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: now also Q4.2 (E), Q8.3 (C)
- net at C2.1, C7.1, R3.1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: now also Q3.3 (C), Q7.2 (E)
- net at R6.1: now also U1.1, U1.3 (+)
- net at R18.2, R19.2: now also U1.2 (-)
- net at R16.2, R17.2: now also U2.6 (-)
- net at R15.1: now also U2.5 (+), U2.7
- net at RV1.2: now also U1.5 (+)
- net at C4.1, R5.1: now also U1.7
- net at R11.2, R7.2: now also Q1.1 (B), Q5.1 (B)
- net at R10.1, R14.2: now also Q4.1 (B), Q8.1 (B)
- net at R12.2, R8.1: now also Q3.1 (B), Q7.1 (B)
- net at R13.2, R9.1: now also Q2.1 (B), Q6.1 (B)
- net at C15.1, R20.1: now also U2.3 (+)
- net at C17.2, C19.2, R24.1: now also U2.1
- net at C17.1, R22.1, R24.2: now also U2.2 (-)
- net at C21.1, R34.1: now also U5.5 (+)
- net at C25.2, R30.1, R38.2: now also U5.6 (-)
- net at R32.2: now also X4.2
- net at R33.2: now also X4.1
- net at C16.1, R21.1: now also U5.3 (+)
- net at C18.2, C20.2, R25.1: now also U5.1
- net at C18.1, R23.1, R25.2: now also U5.2 (-)
- net at C22.1, R35.1: now also U6.5 (+)
- net at C26.2, R31.1, R39.2: now also U6.6 (-)
- net at C27.1, C35.1, C36.1: now also U6.8 (V+), X7.1
- net at JP4.1 (A): now also X7.10
- net at JP5.1 (A): now also X7.12
- net at JP6.1 (A): now also X7.14
- net at C34.1: now also U6.2 (-), X7.2
- net at JP1.1 (A): now also X7.4
- net at JP2.1 (A): now also X7.6
- net at JP3.1 (A): now also X7.8
Other:
- moved on the sheet: C23, C24, C27, C28, C29, C31, C33, C35, C36, JP1, JP2, JP3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
